File: Armor_Plate.kicad_sch (KiCad schematic)
At the start: 46 parts, among them SW3 SW_SP3T

Commit message: Updated fab files
Parts:
- BT1: footprint Battery:BatteryHolder_Keystone_2468_2xAAA -> Battery:BatteryHolder_Keystone_2466_1xAAA
Other:
- note added: "TODO: - Find Specific LED on Mouser - Do Resistance Calculation"
- note removed: "TODO: - Find Specific LED on Mouser - Tie together LED Cathodes - Replace LED Cathode Resistors with singular resistor"
Changed lines of the file:
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@@
 		)
 	)
-	(text "TODO:\n- Find Specific LED on Mouser\n- Tie together LED Cathodes\n- Replace LED Cathode Resistors with singular resistor"
+	(text "TODO:\n- Find Specific LED on Mouser\n- Do Resistance Calculation"
 		(exclude_from_sim no)
 		(at 34.798 75.692 0)
@@
 					(size 1.27 1.27)
 				)
+				(hide yes)
 			)
 		)
@@
 			)
 		)
-		(property "Footprint" "Battery:BatteryHolder_Keystone_2468_2xAAA"
+		(property "Footprint" "Battery:BatteryHolder_Keystone_2466_1xAAA"
 			(at 27.94 112.776 90)
 			(effects

Commit message: Staged for further work by armor plate team
Other:
- note added: "TODO: - Find Specific LEDs on Mouser (0603 package, Red/Blue) - Using LED operating point, determine a good power rail voltage - Do Resistance Calculations - BOM (Mouser Links)"
- note removed: "TODO: - Find Specific LED on Mouser - Do Resistance Calculation"
Changed lines of the file:
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@@
 		)
 	)
-	(text "TODO:\n- Find Specific LED on Mouser\n- Do Resistance Calculation"
+	(text "TODO:\n- Find Specific LEDs on Mouser (0603 package, Red/Blue)\n- Using LED operating point, determine a good power rail voltage\n- Do Resistance Calculations\n- BOM (Mouser Links)"
 		(exclude_from_sim no)
 		(at 34.798 75.692 0)

Commit message: Updated Armor Plate 2 batteries
Parts:
- BT1: footprint Battery:BatteryHolder_Keystone_2466_1xAAA -> Battery:BatteryHolder_Keystone_2468_2xAAA
Changed lines of the file:
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@@
 			)
 		)
-		(property "Footprint" "Battery:BatteryHolder_Keystone_2466_1xAAA"
+		(property "Footprint" "Battery:BatteryHolder_Keystone_2468_2xAAA"
 			(at 27.94 112.776 90)
 			(effects

Commit message: Changed battery cell footprint to hold 3 batteries
Parts:
- BT1: footprint Battery:BatteryHolder_Keystone_2468_2xAAA -> Battery:BatteryHolder_Keystone_2479_3xAAA
Changed lines of the file:
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@@
 			)
 		)
-		(property "Footprint" "Battery:BatteryHolder_Keystone_2468_2xAAA"
+		(property "Footprint" "Battery:BatteryHolder_Keystone_2479_3xAAA"
 			(at 27.94 112.776 90)
 			(effects
